Commit message: Gotowe

File: urdf/my_robot.urdf.xacro (robot description, xacro)
@@ -26,4 +26,21 @@
     </visual>
   </link>
+  <link name="front_marker_link">
+    <visual>
+      <geometry>
+        <box size="0.05 0.02 0.01"/>
+      </geometry>
+      <origin xyz="0 0 0" rpy="0 0 0"/>
+      <material name="black">
+        <color rgba="0 0 0 1"/>
+      </material>
+    </visual>
+  </link>
+    <!-- Złącze do etykiety FRONT -->
+  <joint name="front_marker_joint" type="fixed">
+    <parent link="base_link"/>
+    <child link="front_marker_link"/>
+    <origin xyz="0 -0.087 0.03" rpy="0 0 0"/>
+  </joint>
 <!-- Złącze 1: Obrót bazy -->
   <joint name="base_to_link1" type="revolute">
@@ -48,5 +65,5 @@
       <child link="link2"/>
       <axis xyz="1 0 0"/>
-      <limit lower="-1.5708" upper="1.5708" effort="100" velocity="1.0"/>
+      <limit lower="0" upper="1.4835" effort="100" velocity="1.0"/>
       <origin xyz="0 0 0.044" rpy="0.78 0 0"/>
     </joint>
@@ -66,5 +83,5 @@
       <child link="link3"/>
       <axis xyz="1 0 0"/>
-      <limit lower="-1.5708" upper="1.5708" effort="100" velocity="1.0"/>
+      <limit lower="-0.1745" upper="1.5708" effort="100" velocity="1.0"/>
       <origin xyz="0 0 0.135" rpy="0.78 0 0"/>
     </joint>
@@ -115,3 +132,26 @@
     </visual>
   </link>
+    <link name="silownik">
+    <visual>
+      <geometry>
+        <box size="0.01 0.01 0.03"/>
+      </geometry>
+      <origin xyz="0 0 0" rpy="0 0 0"/>
+      <material name="black">
+        <color rgba="0 0 0 1"/>
+      </material>
+    </visual>
+  </link>
+    <!-- Złącze do etykiety FRONT -->
+  <joint name="silownik_joint" type="fixed">
+    <parent link="link5"/>
+    <child link="silownik"/>
+    <origin xyz="0.02 0.01 -0.015" rpy="0 0 0"/>
+  </joint>
+  <link name="tool_frame" />
+  <joint name="tool_frame_joint" type="fixed">
+    <parent link="link5"/>
+    <child link="tool_frame"/>
+    <origin xyz="0 0 0.01" rpy="0 0 0"/> <!-- przesunięcie np. 10 cm do przodu -->
+  </joint>
 </robot>
